File: QN-hw.kicad_pcb (KiCad board)
At the start: 2 copper layers, 101.6 x 53.3 mm, 13 parts, among them P1 Digital, P10 CONN_01X01, P11 CONN_01X01, P12 CONN_01X01, P13 CONN_01X01, P2 Power, P3 Analog, P4 Analog, P5 PWM, P6 PWM, P7 Communication, P8 CONN_01X01, P9 CONN_01X01

Commit message: schamatic
Parts:
- removed P1: Digital, Socket_Arduino_Mega:Socket_Strip_Arduino_2x18
- removed P2: Power, Socket_Arduino_Mega:Socket_Strip_Arduino_1x08
- removed P3, P4: Analog, Socket_Arduino_Mega:Socket_Strip_Arduino_1x08
- removed P5: PWM, Socket_Arduino_Mega:Socket_Strip_Arduino_1x10
- removed P6: PWM, Socket_Arduino_Mega:Socket_Strip_Arduino_1x08
- removed P7: Communication, Socket_Arduino_Mega:Socket_Strip_Arduino_1x08
- added C1: 1uF, Capacitors_SMD:C_0805, F.Cu at (270.3, 247.9)
- added C10: 1uF, Capacitors_SMD:C_0805, F.Cu at (294.6, 253.0)
- added C11: 1uF, Capacitors_SMD:C_0805, F.Cu at (255.0, 247.9)
- added C12: 1uF, Capacitors_SMD:C_0805, F.Cu at (288.0, 239.3)
- added C13: 1uF, Capacitors_SMD:C_0805, F.Cu at (266.2, 253.0)
- added C14: 1uF, Capacitors_SMD:C_0805, F.Cu at (299.7, 242.3)
- added C15: 1uF, Capacitors_SMD:C_0805, F.Cu at (301.2, 252.0)
- added C16: 1uF, Capacitors_SMD:C_0805, F.Cu at (329.2, 183.4)
- added C17: 1uF, Capacitors_SMD:C_0805, F.Cu at (334.8, 178.8)
- added C18: 1uF, Capacitors_SMD:C_0805, F.Cu at (308.4, 182.9)
- added C19: 1uF, Capacitors_SMD:C_0805, F.Cu at (314.5, 186.9)
- added C2: 1uF, Capacitors_SMD:C_0805, F.Cu at (270.8, 254.0)
- added C20: 1uF, Capacitors_SMD:C_0805, F.Cu at (335.8, 166.6)
- added C21: 0.1uF, Capacitors_SMD:C_0805, F.Cu at (340.9, 158.5)
- added C22: 0.1uF, Capacitors_SMD:C_0805, F.Cu at (287.5, 234.2)
- added C23: 0.1uF, Capacitors_SMD:C_0805, F.Cu at (321.6, 162.6)
- added C24: 0.1uF, Capacitors_SMD:C_0805, F.Cu at (327.7, 176.3)
- added C25: 0.1uF, Capacitors_SMD:C_0805, F.Cu at (304.3, 173.2)
- added C26: 22pF, Capacitors_SMD:C_0805, F.Cu at (299.2, 170.2)
- added C27: 22pF, Capacitors_SMD:C_0805, F.Cu at (321.1, 178.8)
- added C28: 22pF, Capacitors_SMD:C_0805, F.Cu at (328.7, 165.6)
- added C29: 0.1uF, Capacitors_SMD:C_0805, F.Cu at (332.7, 171.2)
- added C3: 1uF, Capacitors_SMD:C_0805, F.Cu at (260.1, 253.5)
- added C4: 1uF, Capacitors_SMD:C_0805, F.Cu at (289.1, 255.5)
- added C5: 1uF, Capacitors_SMD:C_0805, F.Cu at (283.0, 244.9)
- added C6: 1uF, Capacitors_SMD:C_0805, F.Cu at (284.5, 249.9)
- added C7: 1uF, Capacitors_SMD:C_0805, F.Cu at (296.7, 247.4)
- added C8: 1uF, Capacitors_SMD:C_0805, F.Cu at (288.5, 247.4)
- added C9: 1uF, Capacitors_SMD:C_0805, F.Cu at (262.6, 246.9)
- added D1: LED, LEDs:LED_0805, F.Cu at (327.2, 169.2)
- added D10: LED, LEDs:LED_0805, F.Cu at (343.9, 173.2)
- added D11: LED, LEDs:LED_0805, F.Cu at (297.7, 163.6)
- added D12: LED, LEDs:LED_0805, F.Cu at (301.8, 178.8)
- added D13: LED, LEDs:LED_0805, F.Cu at (308.9, 178.8)
- added D14: LED, LEDs:LED_0805, F.Cu at (315.0, 179.3)
- added D15, D17, D19, D6, D8, D9: LED, LEDs:LED_0805, F.Cu at (315.1, 171.6)
- added D16: LED, LEDs:LED_0805, F.Cu at (322.1, 172.2)
- added D18: LED, LEDs:LED_0805, F.Cu at (303.3, 185.9)
- added D2: LED, LEDs:LED_0805, F.Cu at (357.1, 157.0)
- added D20: LED, LEDs:LED_0805, F.Cu at (324.6, 187.5)
- added D21: D, DO-214AC(SMA):DO-214AC(SMA), F.Cu at (256.5, 239.3)
- added D22: D, DO-214AC(SMA):DO-214AC(SMA), F.Cu at (278.9, 239.8)
- added D23: D, DO-214AC(SMA):DO-214AC(SMA), F.Cu at (300.2, 232.2)
- added D24: D, DO-214AC(SMA):DO-214AC(SMA), F.Cu at (279.9, 226.6)
- added D25: D, DO-214AC(SMA):DO-214AC(SMA), F.Cu at (254.5, 231.6)
- added D26: D, DO-214AC(SMA):DO-214AC(SMA), F.Cu at (140.7, 115.8)
- added D27: D, DO-214AC(SMA):DO-214AC(SMA), F.Cu at (141.7, 104.6)
- added D28: D, DO-214AC(SMA):DO-214AC(SMA), F.Cu at (254.0, 223.0)
- added D29: D, DO-214AC(SMA):DO-214AC(SMA), F.Cu at (293.1, 227.1)
- added D3: LED, LEDs:LED_0805, F.Cu at (314.5, 164.1)
- added D30: D, DO-214AC(SMA):DO-214AC(SMA), F.Cu at (295.7, 237.7)
- added D31: D, DO-214AC(SMA):DO-214AC(SMA), F.Cu at (283.5, 220.0)
- added D32: D, DO-214AC(SMA):DO-214AC(SMA), F.Cu at (269.7, 217.4)
- added D33: D, DO-214AC(SMA):DO-214AC(SMA), F.Cu at (265.7, 225.0)
- added D34: D, DO-214AC(SMA):DO-214AC(SMA), F.Cu at (264.7, 233.2)
- added D35: D, DO-214AC(SMA):DO-214AC(SMA), F.Cu at (269.2, 239.3)
- added D36: D, DO-214AC(SMA):DO-214AC(SMA), F.Cu at (293.6, 218.4)
- added D37: D, DO-214AC(SMA):DO-214AC(SMA), F.Cu at (273.3, 221.5)
- added D4: LED, LEDs:LED_0805, F.Cu at (306.3, 163.1)
- added D5: LED, LEDs:LED_0805, F.Cu at (340.9, 189.5)
- added D7: LED, LEDs:LED_0805, F.Cu at (305.3, 167.6)
- added J1: Conn_01x20, Pin_Headers:Pin_Header_Straight_1x20_Pitch2.54mm, F.Cu at (88.9, 76.7)
- added J10: +24V, Pin_Headers:Pin_Header_Angled_1x02_Pitch2.54mm, F.Cu at (154.9, 248.9)
- added J11: Conn_01x02, Pin_Headers:Pin_Header_Angled_1x02_Pitch2.54mm, F.Cu at (156.5, 262.6)
- added J12: Conn_01x02, Pin_Headers:Pin_Header_Angled_1x02_Pitch2.54mm, F.Cu at (178.8, 255.5)
- added J13: Conn_01x02, Pin_Headers:Pin_Header_Angled_1x02_Pitch2.54mm, F.Cu at (138.7, 261.6)
- added J14: Conn_01x02, Pin_Headers:Pin_Header_Angled_1x02_Pitch2.54mm, F.Cu at (179.3, 242.3)
- added J15: Conn_01x02, Pin_Headers:Pin_Header_Angled_1x02_Pitch2.54mm, F.Cu at (171.7, 232.7)
- added J16: Conn_01x02, Pin_Headers:Pin_Header_Angled_1x02_Pitch2.54mm, F.Cu at (170.2, 220.5)
- added J17: Conn_01x02, Pin_Headers:Pin_Header_Angled_1x02_Pitch2.54mm, F.Cu at (206.2, 232.2)
- added J18: Conn_01x02, Pin_Headers:Pin_Header_Angled_1x02_Pitch2.54mm, F.Cu at (150.9, 216.9)
- added J19: Conn_01x02, Pin_Headers:Pin_Header_Angled_1x02_Pitch2.54mm, F.Cu at (193.0, 226.6)
- added J2: +24V, Pin_Headers:Pin_Header_Angled_1x02_Pitch2.54mm, F.Cu at (138.2, 239.3)
- added J20: Conn_01x02, Pin_Headers:Pin_Header_Angled_1x02_Pitch2.54mm, F.Cu at (193.5, 237.2)
- added J21: Conn_01x02, Pin_Headers:Pin_Header_Angled_1x02_Pitch2.54mm, F.Cu at (199.1, 248.4)
- added J3: Boot -loader, Pin_Headers:Pin_Header_Angled_1x06_Pitch2.54mm, F.Cu at (120.9, 105.2)
- added J4: Nap-CT, Pin_Headers:Pin_Header_Angled_1x05_Pitch2.54mm, F.Cu at (119.9, 128.0)
- added J5: Conn_01x02, Pin_Headers:Pin_Header_Angled_1x02_Pitch2.54mm, F.Cu at (177.3, 265.2)
- added J6: Conn_01x02, Pin_Headers:Pin_Header_Angled_1x02_Pitch2.54mm, F.Cu at (137.7, 249.9)
- added J7: Conn_01x02, Pin_Headers:Pin_Header_Angled_1x02_Pitch2.54mm, F.Cu at (136.1, 228.6)
- added J8: Conn_01x02, Pin_Headers:Pin_Header_Angled_1x02_Pitch2.54mm, F.Cu at (149.4, 226.6)
- added J9: Conn_01x02, Pin_Headers:Pin_Header_Angled_1x02_Pitch2.54mm, F.Cu at (153.9, 236.2)
- added Q1, Q10, Q11, Q12, Q13, Q14, Q15, Q16, Q2, Q3, Q4, Q6, Q7, Q8, Q9: Q_NMOS_DGS, TO_SOT_Packages_SMD:SOT-23, F.Cu at (315.1, 171.6)
- added Q5: Q_NMOS_DGS, TO_SOT_Packages_SMD:SOT-23, F.Cu at (342.9, 166.1)
- added R1: 3K3/0.6W, Resistors_THT:R_Axial_DIN0204_L3.6mm_D1.6mm_P5.08mm_Horizontal, F.Cu at (147.3, 127.5)
- added R10: 3K3/0.6W, Resistors_THT:R_Axial_DIN0204_L3.6mm_D1.6mm_P5.08mm_Horizontal, F.Cu at (150.9, 112.3)
- added R100, R101, R102, R103, R107, R120, R121, R122, R123, R124, R125, R144, R81, R82, R83, R84: 220R, Resistors_SMD:R_0805, F.Cu at (315.1, 171.6)
- added R104, R108, R111, R114, R117, R126, R129, R132, R135, R138, R141, R145, R43, R44, R45, R46, R47, R48, R49, R50, R51, R52, R53, R54, R55, R56, R57, R58, R59, R60, R85, R88, R91, R94, R97: 10K, Resistors_SMD:R_0805, F.Cu at (315.1, 171.6)
- added R105, R109, R112, R115, R118, R127, R130, R133, R136, R139, R142, R146, R86, R89, R92, R95, R98: 1K, Resistors_SMD:R_0805, F.Cu at (315.1, 171.6)
- added R106, R110, R113, R116, R119, R128, R131, R134, R137, R140, R143, R147, R90, R93, R96, R99: 10R, Resistors_SMD:R_0805, F.Cu at (315.1, 171.6)
- added R11: 3K3/0.6W, Resistors_THT:R_Axial_DIN0204_L3.6mm_D1.6mm_P5.08mm_Horizontal, F.Cu at (149.4, 137.7)
- added R12: 3K3/0.6W, Resistors_THT:R_Axial_DIN0204_L3.6mm_D1.6mm_P5.08mm_Horizontal, F.Cu at (138.2, 140.2)
- added R13: 3K3/0.6W, Resistors_THT:R_Axial_DIN0204_L3.6mm_D1.6mm_P5.08mm_Horizontal, F.Cu at (154.9, 133.1)
- added R14: 3K3/0.6W, Resistors_THT:R_Axial_DIN0204_L3.6mm_D1.6mm_P5.08mm_Horizontal, F.Cu at (158.0, 105.2)
- added R15: 3K3/0.6W, Resistors_THT:R_Axial_DIN0204_L3.6mm_D1.6mm_P5.08mm_Horizontal, F.Cu at (141.7, 133.6)
- added R16: 3K3/0.6W, Resistors_THT:R_Axial_DIN0204_L3.6mm_D1.6mm_P5.08mm_Horizontal, F.Cu at (145.3, 148.3)
- added R17: 3K3/0.6W, Resistors_THT:R_Axial_DIN0204_L3.6mm_D1.6mm_P5.08mm_Horizontal, F.Cu at (148.3, 120.4)
- added R18: 3K3/0.6W, Resistors_THT:R_Axial_DIN0204_L3.6mm_D1.6mm_P5.08mm_Horizontal, F.Cu at (133.6, 157.0)
- added R19: 3K3/0.6W, Resistors_THT:R_Axial_DIN0204_L3.6mm_D1.6mm_P5.08mm_Horizontal, F.Cu at (151.4, 159.5)
- added R2: 3K3/0.6W, Resistors_THT:R_Axial_DIN0204_L3.6mm_D1.6mm_P5.08mm_Horizontal, F.Cu at (147.3, 111.8)
- added R20: 3K3/0.6W, Resistors_THT:R_Axial_DIN0204_L3.6mm_D1.6mm_P5.08mm_Horizontal, F.Cu at (134.1, 148.3)
- added R21: 1K/0.6W, Resistors_THT:R_Axial_DIN0204_L3.6mm_D1.6mm_P5.08mm_Horizontal, F.Cu at (156.0, 152.9)
- added R22: 1K/0.6W, Resistors_THT:R_Axial_DIN0204_L3.6mm_D1.6mm_P5.08mm_Horizontal, F.Cu at (144.3, 155.4)
- added R23, R24, R25, R26, R27, R28, R29, R30, R31, R32, R33, R34, R35, R36, R37, R38, R39, R40: 1K/0.6W, Resistors_THT:R_Axial_DIN0204_L3.6mm_D1.6mm_P5.08mm_Horizontal, F.Cu at (148.5, 105.0)
- added R3: 3K3/0.6W, Resistors_THT:R_Axial_DIN0204_L3.6mm_D1.6mm_P5.08mm_Horizontal, F.Cu at (146.8, 111.8)
- added R4: 3K3/0.6W, Resistors_THT:R_Axial_DIN0204_L3.6mm_D1.6mm_P5.08mm_Horizontal, F.Cu at (149.4, 100.1)
- added R41: 10K, Resistors_SMD:R_0805, F.Cu at (277.9, 249.4)
- added R42: 10K, Resistors_SMD:R_0805, F.Cu at (280.9, 254.5)
- added R5: 3K3/0.6W, Resistors_THT:R_Axial_DIN0204_L3.6mm_D1.6mm_P5.08mm_Horizontal, F.Cu at (146.8, 100.1)
- added R6: 3K3/0.6W, Resistors_THT:R_Axial_DIN0204_L3.6mm_D1.6mm_P5.08mm_Horizontal, F.Cu at (158.5, 101.6)
- added R61, R62, R63, R64, R65, R66, R67, R68, R69, R70, R71, R72, R73, R74, R75, R76, R77, R78, R79, R80: 220R/0.6W, Resistors_THT:R_Axial_DIN0204_L3.6mm_D1.6mm_P5.08mm_Horizontal, F.Cu at (148.5, 105.0)
- added R7: 3K3/0.6W, Resistors_THT:R_Axial_DIN0204_L3.6mm_D1.6mm_P5.08mm_Horizontal, F.Cu at (159.5, 110.2)
- added R8: 3K3/0.6W, Resistors_THT:R_Axial_DIN0204_L3.6mm_D1.6mm_P5.08mm_Horizontal, F.Cu at (160.0, 117.3)
- added R87: 1M, Resistors_SMD:R_0805, F.Cu at (315.1, 171.6)
- added R9: 3K3/0.6W, Resistors_THT:R_Axial_DIN0204_L3.6mm_D1.6mm_P5.08mm_Horizontal, F.Cu at (156.5, 124.5)
- added SW1: SW_Push, Buttons_Switches_SMD:SW_DIP_x1_W5.08mm_Slide_Copal_CHS-A, F.Cu at (140.2, 109.7)
- added U1: TLP627-4, Housings_DIP:DIP-16_W7.62mm, F.Cu at (191.5, 86.9)
- added U10: ATMEGA2560-16AU, Housings_QFP:LQFP-100_14x14mm_Pitch0.5mm, F.Cu at (131.6, 80.8)
- added U11: TLP627-4, Housings_DIP:DIP-16_W7.62mm, F.Cu at (234.2, 93.0)
- added U12: TLP627-4, Housings_DIP:DIP-16_W7.62mm, F.Cu at (259.1, 136.1)
- added U13: TLP627-4, Housings_DIP:DIP-16_W7.62mm, F.Cu at (269.2, 41.1)
- added U14: TLP627-4, Housings_DIP:DIP-16_W7.62mm, F.Cu at (188.5, 117.3)
- added U2: TLP627-4, Housings_DIP:DIP-16_W7.62mm, F.Cu at (182.4, 61.5)
- added U3: TLP627-4, Housings_DIP:DIP-16_W7.62mm, F.Cu at (174.2, 117.3)
- added U4: TLP627-4, Housings_DIP:DIP-16_W7.62mm, F.Cu at (173.7, 86.4)
- added U5: TLP627-4, Housings_DIP:DIP-16_W7.62mm, F.Cu at (168.7, 61.0)
- added U6: 74HC14, Housings_DIP:DIP-14_W7.62mm, F.Cu at (166.6, 25.4)
- added U7: 74HC14, Housings_DIP:DIP-14_W7.62mm, F.Cu at (199.6, 30.0)
- added U8: 74HC14, Housings_DIP:DIP-14_W7.62mm, F.Cu at (214.9, 122.4)
- added U9: 74HC14, Housings_DIP:DIP-14_W7.62mm, F.Cu at (269.2, 94.5)
- added Y1: 20Mhz, Crystals:Crystal_SMD_HC49-SD, F.Cu at (130.6, 96.0)
- P10, P11, P12, P13, P8, P9: footprint Socket_Arduino_Mega:Arduino_1pin -> Pin_Headers:Pin_Header_Angled_1x01_Pitch2.54mm
- moved P13 274.4 mm to (-6.60, 258.6)
- moved P12 244.1 mm to (-10.2, 251.5)
- moved P10 240.5 mm to (-9.65, 237.2)
- moved P11 216.2 mm to (-9.65, 244.9)
- moved P9 212.5 mm to (-10.2, 227.6)
- moved P8 170.4 mm to (-10.2, 232.2)
Connections:
- P10 pad 1: Net-(P10-Pad1) -> (no net)
- P11 pad 1: Net-(P11-Pad1) -> (no net)
- P12 pad 1: Net-(P12-Pad1) -> (no net)
- P13 pad 1: Net-(P13-Pad1) -> (no net)
- P8 pad 1: Net-(P8-Pad1) -> (no net)
- P9 pad 1: Net-(P9-Pad1) -> (no net)
Other:
- board outline removed
- board text removed: "1"
