File: QN-hw.kicad_pcb (KiCad board)
At the start: 2 copper layers, 272 parts, among them J1 Conn_01x20, J10 +24V, J11 Conn_01x02, J12 Conn_01x02, J13 Conn_01x02, J14 Conn_01x02, J15 Conn_01x02, J16 Conn_01x02, J17 Conn_01x02, J18 Conn_01x02, J19 Conn_01x02, J2 +24V, J20 Conn_01x02, J21 Conn_01x02, J3 Boot -loader, J4 Nap-CT, J5 Conn_01x02, J6 Conn_01x02, J7 Conn_01x02, J8 Conn_01x02, J9 Conn_01x02, P10 CONN_01X01, P11 CONN_01X01, P12 CONN_01X01, P13 CONN_01X01, P8 CONN_01X01, P9 CONN_01X01, Q1 Q_NMOS_DGS, Q10 Q_NMOS_DGS, Q11 Q_NMOS_DGS, Q12 Q_NMOS_DGS, Q13 Q_NMOS_DGS, Q14 Q_NMOS_DGS, Q15 Q_NMOS_DGS, Q16 Q_NMOS_DGS, Q2 Q_NMOS_DGS, Q3 Q_NMOS_DGS, Q4 Q_NMOS_DGS, Q5 Q_NMOS_DGS, Q6 Q_NMOS_DGS, Q7 Q_NMOS_DGS, Q8 Q_NMOS_DGS, Q9 Q_NMOS_DGS, SW1 SW_Push, U1 TLP627-4, U10 ATMEGA2560-16AU, U11 TLP627-4, U12 TLP627-4, U13 TLP627-4, U14 TLP627-4, U2 TLP627-4, U3 TLP627-4, U4 TLP627-4, U5 TLP627-4, U6 74HC14, U7 74HC14, U8 74HC14, U9 74HC14, Y1 20Mhz

Commit message: sap xep linh kien
Parts:
- R1, R10, R11, R12, R13, R14, R15, R16, R17, R18, R19, R2, R20, R21, R22, R23, R24, R25, R26, R27, R28, R29, R3, R30, R31, R32, R33, R34, R35, R36, R37, R38, R39, R4, R40, R5, R6, R7, R8, R9: footprint Resistors_THT:R_Axial_DIN0204_L3.6mm_D1.6mm_P5.08mm_Horizontal -> Resistors_SMD:R_2512
- R108, R111, R114, R117, R126, R129, R132, R135, R138, R141, R145, R88, R91, R94, R97: value 10K -> 10K/0.6W; footprint Resistors_SMD:R_0805 -> Resistors_SMD:R_2512
- R109, R112, R115, R118, R127, R130, R133, R136, R139, R142, R146, R89, R92, R95, R98: value 1K -> 1K/0.6W; footprint Resistors_SMD:R_0805 -> Resistors_SMD:R_2512
- R110, R113, R116, R119, R128, R131, R134, R137, R140, R143, R90, R93, R96, R99: value 10R -> 10R/0.6W; footprint Resistors_SMD:R_0805 -> Resistors_SMD:R_2512
- R147: value 10R -> 10/R0.6W; footprint Resistors_SMD:R_0805 -> Resistors_SMD:R_2512
- R61, R62, R63, R64, R65, R66, R67, R68, R69, R70, R71, R72, R73, R74, R75, R76, R77, R78, R79, R80: value 220R/0.6W -> 220R; footprint Resistors_THT:R_Axial_DIN0204_L3.6mm_D1.6mm_P5.08mm_Horizontal -> Resistors_SMD:R_0805
- moved J4 267.9 mm to (386.1, 97.8)
- moved U10 254.4 mm to (381.0, 130.8)
- moved J3 242.6 mm to (363.2, 92.7)
- moved Y1 231.6 mm to (356.4, 147.3), turned to 90 degrees
- moved R141 219.1 mm to (111.8, 89.9)
- moved R121 212.5 mm to (116.3, 96.5)
- moved R140 211.9 mm to (122.9, 82.3)
- moved R120 208.8 mm to (122.9, 89.9)
- moved R139 207.5 mm to (130.6, 76.7)
- moved R122 206.2 mm to (120.4, 103.6)
- moved Q16 206.1 mm to (110.2, 149.4)
- moved R95 205.5 mm to (110.2, 155.4)
- moved R102 204.4 mm to (110.7, 172.7)
- moved R94 203.5 mm to (111.8, 164.1)
- moved R125 202.8 mm to (131.1, 86.4)
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Connections:
- R79 pad 1: (no net) -> GND

Commit message: complete
Parts:
- removed P10, P12: CONN_01X01, Pin_Headers:Pin_Header_Angled_1x01_Pitch2.54mm
- added J22: +5V, Termical-block-2:Pin_Header_Angled_1x02_Pitch2.54mm, F.Cu at (290.7, 115.7)
- added J24: I2C, nhantt-kicad-lib:Pin_Header_Straight_1x04_Pitch2.54mm, F.Cu at (399.2, 112.5)
- added J25: I2C, nhantt-kicad-lib:Pin_Header_Straight_1x04_Pitch2.54mm, F.Cu at (403.7, 112.5)
- added J26: ADC-5V, nhantt-kicad-lib:Pin_Header_Straight_1x10_Pitch2.54mm, F.Cu at (365.5, 119.5)
- added J27: UART, nhantt-kicad-lib:Pin_Header_Straight_1x08_Pitch2.54mm, F.Cu at (370.3, 112.4)
- added P1: CONN_01X01, nhantt-kicad-lib:Vit-3mm, F.Cu at (355.6, 241.3)
- added P2: CONN_01X01, nhantt-kicad-lib:Vit-3mm, F.Cu at (355.6, 111.8)
- added R148: 10K/0.6W, Resistors_SMD:R_0805, F.Cu at (413.8, 212.0)
- added R149: 10K/0.6W, Resistors_SMD:R_0805, F.Cu at (410.8, 215.2)
- added R150: 10K/0.6W, Resistors_SMD:R_0805, F.Cu at (397.9, 227.8)
- added R151: 10K/0.6W, Resistors_SMD:R_0805, F.Cu at (414.3, 223.5)
- added R152: 10K/0.6W, Resistors_SMD:R_0805, F.Cu at (413.8, 204.5)
- added R153: 10K/0.6W, Resistors_SMD:R_0805, F.Cu at (409.3, 126.2)
- added R154: 10K/0.6W, Resistors_SMD:R_0805, F.Cu at (410.7, 121.5)
- added R155: 10K/0.6W, Resistors_SMD:R_0805, F.Cu at (410.5, 116.5)
- added R156: 10K/0.6W, Resistors_SMD:R_0805, F.Cu at (410.5, 163.2)
- added R157: 10K/0.6W, Resistors_SMD:R_0805, F.Cu at (413.5, 170.4)
- added R158: 10K/0.6W, Resistors_SMD:R_0805, F.Cu at (411.5, 177.4)
- added R159: 10K, Resistors_SMD:R_0805, F.Cu at (415.3, 160.1)
- added R160: 10K/0.6W, Resistors_SMD:R_0805, F.Cu at (410.2, 111.4)
- added R161: 10K/0.6W, Resistors_SMD:R_0805, F.Cu at (413.4, 197.0)
- added R162: 10K/0.6W, Resistors_SMD:R_0805, F.Cu at (415.5, 191.6)
- added R163: 10K/0.6W, Resistors_SMD:R_0805, F.Cu at (410.7, 185.9)
- J1: footprint Pin_Headers:Pin_Header_Straight_1x20_Pitch2.54mm -> mods:Terminal-block-20
- J10, J11, J12, J13, J14, J15, J16, J17, J18, J19, J2, J20, J21, J5, J6, J7, J8, J9: footprint Pin_Headers:Pin_Header_Angled_1x02_Pitch2.54mm -> Termical-block-2:Pin_Header_Angled_1x02_Pitch2.54mm
- P11, P13, P8, P9: footprint Pin_Headers:Pin_Header_Angled_1x01_Pitch2.54mm -> nhantt-kicad-lib:Vit-3mm
- R108, R109, R110, R111, R112, R113, R114, R115, R116, R117, R118, R119, R126, R127, R128, R129, R130, R131, R132, R133, R134, R135, R136, R137, R138, R139, R140, R141, R142, R143, R145, R146, R147, R88, R89, R90, R91, R92, R93, R94, R95, R96, R97, R98, R99: footprint Resistors_SMD:R_2512 -> Resistors_SMD:R_0805
- U10: footprint Housings_QFP:LQFP-100_14x14mm_Pitch0.5mm -> Housings_QFP:TQFP-100_14x14mm_Pitch0.5mm
- moved P8 460.5 mm to (434.3, 111.8)
- moved P9 447.2 mm to (436.9, 240.0)
- moved D27 441.9 mm to (421.5, 112.5)
- moved D26 440.9 mm to (419.9, 157.4), turned to 180 degrees
- moved D28 395.5 mm to (421.5, 117.7)
- moved SW1 367.0 mm to (345.4, 127.0), turned to 270 degrees
- moved D34 362.3 mm to (420.1, 182.6), turned to 180 degrees
- moved R37 361.6 mm to (316.2, 219.7), turned to 180 degrees
- moved D30 361.4 mm to (421.5, 127.6)
- moved D33 361.0 mm to (419.9, 175.2), turned to 180 degrees
- moved D29 360.8 mm to (421.6, 122.6)
- moved D25 359.8 mm to (420.9, 227.2), turned to 180 degrees
- moved R38 358.3 mm to (316.2, 226.1), turned to 180 degrees
- moved D35 358.2 mm to (420.3, 189.0), turned to 180 degrees
- moved D32 356.7 mm to (419.9, 168.8), turned to 180 degrees
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Connections:
- J3 pad 1: VCC -> GND
- J3 pad 2: GND -> VCC
- J4 pad 1: VCC -> GND
- J4 pad 2: GND -> VCC
- Q7 pad 3: Net-(Q7-Pad3) -> /0V-OUT
- R102 pad 1: 31 -> 24
- R103 pad 1: 36 -> 25
- R106 pad 2: Net-(R104-Pad2) -> Net-(R106-Pad2)
- R107 pad 1: 34 -> 26
- R110 pad 2: Net-(R108-Pad2) -> Net-(R110-Pad2)
- R113 pad 2: Net-(R111-Pad2) -> Net-(R113-Pad2)
- R116 pad 2: Net-(R114-Pad2) -> Net-(R116-Pad2)
- R119 pad 2: Net-(R117-Pad2) -> Net-(R119-Pad2)
- R120 pad 1: 25 -> 27
- R121 pad 1: 26 -> 28
- R122 pad 1: 27 -> 29
- R123 pad 1: 28 -> 30
- R124 pad 1: 29 -> 31
- R125 pad 1: 24 -> 32
- R128 pad 2: Net-(R126-Pad2) -> Net-(R128-Pad2)
- R131 pad 2: Net-(R129-Pad2) -> Net-(R131-Pad2)
- R134 pad 2: Net-(R132-Pad2) -> Net-(R134-Pad2)
- R137 pad 2: Net-(R135-Pad2) -> Net-(R137-Pad2)
- R140 pad 2: Net-(R138-Pad2) -> Net-(R140-Pad2)
- R143 pad 2: Net-(R141-Pad2) -> Net-(R143-Pad2)
- R147 pad 2: Net-(R145-Pad2) -> Net-(R147-Pad2)
- R41 pad 2: 1 -> I1
- R42 pad 2: 2 -> I2
- R43 pad 2: 3 -> I3
- R44 pad 2: 4 -> I4
- R45 pad 2: 5 -> I5
- R46 pad 2: 8 -> I8
- R47 pad 2: 6 -> I6
- R48 pad 2: 7 -> I7
- R49 pad 2: 9 -> I9
- R50 pad 2: 10 -> I10
- R51 pad 2: 11 -> I11
- R52 pad 2: 12 -> I12
- R53 pad 2: 13 -> I13
- R54 pad 2: 14 -> I14
- R55 pad 2: 15 -> I15
- R56 pad 2: 16 -> I16
- R57 pad 2: 17 -> I17
- R58 pad 2: 18 -> I18
- R59 pad 2: 19 -> I19
- R60 pad 2: 20 -> I20
- R81 pad 1: 37 -> 34
- R82 pad 1: 30 -> 44
- R83 pad 1: 35 -> 45
- R84 pad 1: 32 -> 48
- R90 pad 2: Net-(R88-Pad2) -> Net-(R148-Pad2)
- R93 pad 2: Net-(R91-Pad2) -> Net-(R149-Pad2)
- R96 pad 2: Net-(R94-Pad2) -> Net-(R151-Pad2)
- R99 pad 2: Net-(R97-Pad2) -> Net-(R150-Pad2)
- U1 pad 10: 16 -> I16
- U1 pad 12: 15 -> I15
- U1 pad 14: 14 -> I14
- U1 pad 16: 13 -> I13
- U10 pad 12: (no net) -> RX2
- U10 pad 13: (no net) -> TX2
- U10 pad 43: (no net) -> SCL
- U10 pad 44: (no net) -> SDA
- U10 pad 45: (no net) -> RX1
- U10 pad 46: (no net) -> TX1
- U10 pad 63: (no net) -> RX3
- U10 pad 64: (no net) -> TX3
- U10 pad 90: (no net) -> A7
- U10 pad 91: (no net) -> A6
- U10 pad 92: (no net) -> A5
- U10 pad 93: (no net) -> A4
- U10 pad 94: (no net) -> A3
- U10 pad 95: (no net) -> A2
- U10 pad 96: (no net) -> A1
- U10 pad 97: (no net) -> A0
- U11 pad 11: /0V-OUT -> Net-(R151-Pad2)
- U11 pad 13: /0V-OUT -> Net-(R149-Pad2)
- U11 pad 15: /0V-OUT -> Net-(R148-Pad2)
- U11 pad 9: /0V-OUT -> Net-(R150-Pad2)
- U12 pad 11: /0V-OUT -> Net-(R116-Pad2)
- U12 pad 13: Net-(Q7-Pad3) -> Net-(R113-Pad2)
- U12 pad 15: /0V-OUT -> Net-(R110-Pad2)
- U12 pad 9: /0V-OUT -> Net-(R119-Pad2)
- U13 pad 11: /0V-OUT -> Net-(R131-Pad2)
- U13 pad 13: /0V-OUT -> Net-(R128-Pad2)
- U13 pad 15: /0V-OUT -> Net-(R106-Pad2)
- U13 pad 9: /0V-OUT -> Net-(R134-Pad2)
- U14 pad 11: /0V-OUT -> Net-(R143-Pad2)
- U14 pad 13: /0V-OUT -> Net-(R140-Pad2)
- U14 pad 15: /0V-OUT -> Net-(R137-Pad2)
- U14 pad 9: /0V-OUT -> Net-(R147-Pad2)
- U2 pad 10: 20 -> I20
- U2 pad 12: 19 -> I19
- U2 pad 14: 18 -> I18
- U2 pad 16: 17 -> I17
- U3 pad 10: 4 -> I4
- U3 pad 12: 3 -> I3
- U3 pad 14: 2 -> I2
- U3 pad 16: 1 -> I1
- U4 pad 10: 8 -> I8
- U4 pad 12: 7 -> I7
- U4 pad 14: 6 -> I6
- U4 pad 16: 5 -> I5
- U5 pad 10: 12 -> I12
- U5 pad 12: 11 -> I11
- U5 pad 14: 10 -> I10
- U5 pad 16: 9 -> I9
- U7 pad 12: 45 -> 36
- U7 pad 8: 48 -> 37
- U8 pad 4: 44 -> 35
Routing:
- net GND: track 0.00 -> 697.6 mm, vias 0 -> 5
- net VCC: track 0.00 -> 597.8 mm, vias 0 -> 5
- net /+24V-OUT: track 0.00 -> 498.4 mm, vias 0 -> 18
- net /0V-OUT: track 0.00 -> 393.0 mm, vias 0 -> 34
- net /0V-IN: track 0.00 -> 390.8 mm
- net 40: track 0.00 -> 102.7 mm, vias 0 -> 2
- net 38: track 0.00 -> 97.6 mm, vias 0 -> 2
- net 35: track 0.00 -> 88.6 mm, vias 0 -> 2
- net 39: track 0.00 -> 83.9 mm, vias 0 -> 1
- net 48: track 0.00 -> 83.2 mm, vias 0 -> 2
- net A10: track 0.00 -> 82.5 mm, vias 0 -> 3
- net Net-(D22-Pad2): track 0.00 -> 81.8 mm, vias 0 -> 1
- net 41: track 0.00 -> 80.8 mm, vias 0 -> 3
- net 43: track 0.00 -> 80.4 mm
- net 42: track 0.00 -> 76.6 mm
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- added copper zone on B.Cu, net /0V-IN
- added copper zone on F.Cu, net /0V-IN
- added copper zone on B.Cu, net /0V-OUT
- added copper zone on F.Cu, net /0V-OUT
- added copper zone on B.Cu, net GND
- added copper zone on F.Cu, net GND
Other:
- board outline added: 156.2 x 135.9 mm
- net class Default: trace_width 0.25 -> 0.2
- net class Source added: clearance 0.2, trace_width 1, via_dia 1.2, via_drill 0.6
