File: QN-hw.sch (KiCad schematic (older format))
At the start: 52 parts, among them P1 Digital, P10 CONN_01X01, P11 CONN_01X01, P12 CONN_01X01, P13 CONN_01X01, P2 Power, P3 Analog, P4 Analog, P5 PWM, P6 PWM, P7 Communication, P8 CONN_01X01, P9 CONN_01X01

Commit message: make input
Parts:
- removed P1: Digital, Socket_Arduino_Mega:Socket_Strip_Arduino_2x18, symbol CONN_02X18
- removed P2: Power, Socket_Arduino_Mega:Socket_Strip_Arduino_1x08, symbol CONN_01X08
- removed P3, P4: Analog, Socket_Arduino_Mega:Socket_Strip_Arduino_1x08, symbol CONN_01X08
- removed P5: PWM, Socket_Arduino_Mega:Socket_Strip_Arduino_1x10, symbol CONN_01X10
- removed P6: PWM, Socket_Arduino_Mega:Socket_Strip_Arduino_1x08, symbol CONN_01X08
- removed P7: Communication, Socket_Arduino_Mega:Socket_Strip_Arduino_1x08, symbol CONN_01X08
- added R? (x14): 1K/0.6W, symbol R
- added R? (x9): 3K3/0.6W, symbol R
- added R? (x20): 10K, symbol R
- added U? (x20): 74HC14, symbol 74HC14
- added U?: ATMEGA2560-16AU, TQFP100, symbol ATMEGA2560-16AU
Connections:
- net labels added: 0V, 1, 10, 11, 12, 13, 14, 15, 16, 17, 18, 19, 2, 20, 3, 4, 5, 6, 7, 8, 9
- net labels removed: +3.3V, 0(Rx0), 1(Tx0), 10(**), 11(**), 12(**), 13(**), 14(Tx3), 15(Rx3), 16(Tx2), 17(Rx2), 18(Tx1), 19(Rx1), 2(**), 20(SDA), 21(SCL), 22, 23, 24, 25, 26, 27, 28, 29, 3(**), 30, 31, 32, 33, 34, 35, 36, 37, 38, 39, 4(**), 40, 41, 42, 43, 44, 45, 46, 47, 48, 49, 5(**), 50(MISO), 51(MOSI), 52(SCK), 53(SS), 6(**), 7(**), 8(**), 9(**), AREF, GND, IOREF, Reset, SCL, SDA, Vin
- wire segments 137 -> 220
- no-connect marks 7 -> 6
Other:
- note removed: "1"
- note removed: "Shield for Arduino Mega Rev 3"
- moved on the sheet: U?A, U?B, U?C, U?D

Commit message: input
Parts:
- added C1, C10, C11, C12, C13, C14, C15, C16, C17, C18, C19, C2, C20, C3, C4, C5, C6, C7, C8, C9: 1uF, symbol C_Small
- added C21, C22, C23, C24, C? (x2): 0.1uF, symbol C
- added C? (x3): 22pF, symbol C
- added D?: D, symbol D
- added J?: Boot -loader, symbol Conn_01x06
- added J?: Nap-CT, symbol Conn_01x05
- added R?: 1M, symbol R
- added R?: 10K, symbol R
- added R?: 1K, symbol R
- added SW?: SW_Push, nhantt-kicad-lib:button-pcb-10mm, symbol SW_Push
- added Y1: 16Mhz, symbol Crystal_GND2
- gave numbers to parts that had none: 72
Connections:
- net +5V is gone; now on net VCC: R41.1, R42.1, R43.1, R44.1, R45.1, R46.1, R47.1, R48.1, R49.1, R50.1, R51.1, R52.1, R53.1, R54.1, R55.1, R56.1, R57.1, R58.1, R59.1, R60.1
- net 0V is gone; now on net GND: U1.11, U1.13, U1.15, U1.9, U2.11, U2.13, U2.15, U2.9, U3.11, U3.13, U3.15, U3.9, U4.11, U4.13, U4.15, U4.9, U5.11, U5.13, U5.15, U5.9
- net 0V-IN: now also C1.2, C10.2, C11.2, C12.2, C13.2, C14.2, C15.2, C16.2, C17.2, C18.2, C19.2, C2.2, C20.2, C3.2, C4.2, C5.2, C6.2, C7.2, C8.2, C9.2
- net 1: now also U6.3; no longer U6.1
- net 12: now also U8.1; no longer U8.13
- net 13: now also U7.13; no longer U7.1
- net 18: now also U9.3; no longer U9.13
- net 19: now also U8.13; no longer U8.1
- net 2: now also U6.1; no longer U6.3
- net 4: now also U6.11; no longer U6.9
- net 5: now also U6.13; no longer U6.11
- net 6: now also U6.9; no longer U6.13
- net A10: now also U6.6
- net A11: now also U6.10
- net A12: now also U6.12
- net A13: now also U6.8
- net A14: now also U7.2
- net A15: now also U7.4
- net A8: now also U6.4
- net A9: now also U6.2
- net GND: now also U10.11 (GND), U10.32 (GND), U10.62 (GND), U10.81 (GND), U10.99 (GND), C21.2, C22.2, C23.2, C24.2, C?.1, C?.2, C?.2, C?.2, J?.2 (Pin_2), J?.2 (Pin_2), R?.1, SW?.2, Y1.2
- net VCC: now also U10.10 (VCC), U10.100 (AVCC), U10.31 (VCC), U10.61 (VCC), U10.80 (VCC), C21.1, C22.1, C23.1, C24.1, D?.1 (K), J?.1 (Pin_1), J?.1 (Pin_1), R?.2
- net at R1.1, R21.2, U3.1: now also C9.1
- net at R2.1, R22.2, U3.3: now also C10.1
- net at R23.2, R3.1, U3.5: now also C11.1
- net at R24.2, R4.1, U3.7: now also C12.1
- net at R25.2, R5.1, U4.1: now also C13.1
- net at R26.2, R6.1, U4.3: now also C14.1
- net at R27.2, R7.1, U4.5: now also C15.1
- net at R28.2, R8.1, U4.7: now also C16.1
- net at R29.2, R9.1, U5.1: now also C17.1
- net at R10.1, R30.2, U5.3: now also C18.1
- net at R11.1, R31.2, U5.5: now also C19.1
- net at R12.1, R32.2, U5.7: now also C20.1
- net at R13.1, R33.2, U1.1: now also C1.1
- net at R14.1, R34.2, U1.3: now also C2.1
- net at R15.1, R35.2, U1.5: now also C3.1
- net at R16.1, R36.2, U1.7: now also C4.1
- net at R17.1, R37.2, U2.1: now also C5.1
- net at R18.1, R38.2, U2.3: now also C6.1
- net at R19.1, R39.2, U2.5: now also C7.1
- net at R20.1, R40.2, U2.7: now also C8.1
- net 49: now reaches U7.6
- net 49: now also U10.35 (PL0(ICP4))
- net 48: now reaches U7.8
- net 48: now also U10.36 (PL1(ICP5))
- net 47: now reaches U7.10
- net 47: now also U10.37 (PL2(T5))
- net 44: now reaches U8.4
- net 44: now also U10.40 (PL5(OC5C))
- net 43: now reaches U8.6
- net 43: now also U10.41 (PL6)
- net 42: now reaches U8.8
- net 42: now also U10.42 (PL7)
- net 41: now reaches U8.10
- net 41: now also U10.51 (PG0(~WR~))
- net 38: now reaches U9.2
- net 38: now also U10.50 ((T2)PD7)
- net RX0: now reaches U10.2 ((PCINT8/RXD0)PE0)
- net RX0: now also J?.4 (Pin_4)
- net SCK: now reaches U10.20 ((PCINT1/SCK)PB1)
- net SCK: now also J?.4 (Pin_4)
- net MOSI: now reaches U10.21 ((PCINT2/MOSI)PB2)
- net MOSI: now also J?.5 (Pin_5)
- net MISO: now reaches U10.22 ((PCINT3/MISO)PB3)
- net MISO: now also J?.6 (Pin_6)
- net TX0: now reaches U10.3 ((TXD0)PE1)
- net TX0: now also J?.5 (Pin_5)
- net RST: now reaches U10.30 (~RESET)
- net RST: now also C?.1, C?.2, D?.2 (A), J?.3 (Pin_3), R?.1, SW?.1
- net at U10.33 (XTAL2): now also C?.2, R?.2, Y1.1
- net at U10.34 (XTAL1): now also C?.1, R?.1, Y1.3
- net 46: now reaches U10.38 (PL3(OC5A))
- net 46: now also U8.2
- net 45: now reaches U10.39 (PL4(OC5B))
- net 45: now also U7.12
- net 40: now reaches U10.52 (PG1(~RD~))
- net 40: now also U9.4
- net 39: now reaches U10.70 (PG2(ALE))
- net 39: now also U8.12
- net at U10.98 (AREF): now also C?.1
- new net DTR: C?.1, J?.3 (Pin_3), R?.2

Commit message: schamatic
Parts:
- removed Y1: 16Mhz, symbol Crystal_GND2
- added D1, D10, D11, D12, D13, D14, D15, D16, D17, D18, D19, D2, D20, D3, D4, D5, D6, D7, D8, D9: LED, LEDs:LED_0805, symbol LED
- added D22, D23, D24, D25, D26, D27, D28, D29, D30, D31, D32, D33, D34, D35, D36, D37: D, DO-214AC(SMA):DO-214AC(SMA), symbol D
- added J10: +24V, Pin_Headers:Pin_Header_Angled_1x02_Pitch2.54mm, symbol Conn_01x02
- added J11, J12, J13, J14, J15, J16, J17, J18, J19, J20, J21, J5, J6, J7, J8, J9: Conn_01x02, Pin_Headers:Pin_Header_Angled_1x02_Pitch2.54mm, symbol Conn_01x02
- added Q1, Q10, Q11, Q12, Q13, Q14, Q15, Q16, Q2, Q3, Q4, Q5, Q6, Q7, Q8, Q9: Q_NMOS_DGS, TO_SOT_Packages_SMD:SOT-23, symbol Q_NMOS_DGS
- added R100, R101, R102, R103, R107, R120, R121, R122, R123, R124, R125, R144, R81, R82, R83, R84: 220R, Resistors_SMD:R_0805, symbol R
- added R104, R108, R111, R114, R117, R126, R129, R132, R135, R138, R141, R145, R88, R91, R94, R97: 10K, Resistors_SMD:R_0805, symbol R
- added R105, R109, R112, R115, R118, R127, R130, R133, R136, R139, R142, R146, R89, R92, R95, R98: 1K, Resistors_SMD:R_0805, symbol R
- added R106, R110, R113, R116, R119, R128, R131, R134, R137, R140, R143, R147, R90, R93, R96, R99: 10R, Resistors_SMD:R_0805, symbol R
- added R61, R62, R63, R64, R65, R66, R67, R68, R69, R70, R71, R72, R73, R74, R75, R76, R77, R78, R79, R80: 220R/0.6W, Resistors_THT:R_Axial_DIN0204_L3.6mm_D1.6mm_P5.08mm_Horizontal, symbol R
- added U11, U12, U13, U14: TLP627-4, Housings_DIP:DIP-16_W7.62mm, symbol TLP627-4
- added Y1: 20Mhz, Crystals:Crystal_SMD_HC49-SD, symbol Crystal
- C1, C10, C11, C12, C13, C14, C15, C16, C17, C18, C19, C2, C20, C21, C22, C23, C24, C3, C4, C5, C6, C7, C8, C9: footprint (none) -> Capacitors_SMD:C_0805
- C25, C26, C27, C28, C29: renamed from C?; footprint (none) -> Capacitors_SMD:C_0805
- D21: renamed from D?; footprint (none) -> DO-214AC(SMA):DO-214AC(SMA)
- J1: footprint (none) -> Pin_Headers:Pin_Header_Straight_1x20_Pitch2.54mm
- J2: footprint (none) -> Pin_Headers:Pin_Header_Angled_1x02_Pitch2.54mm
- J3: renamed from J?; footprint (none) -> Pin_Headers:Pin_Header_Angled_1x06_Pitch2.54mm
- J4: renamed from J?; footprint (none) -> Pin_Headers:Pin_Header_Angled_1x05_Pitch2.54mm
- P10, P11, P12, P13, P8, P9: footprint Socket_Arduino_Mega:Arduino_1pin -> Pin_Headers:Pin_Header_Angled_1x01_Pitch2.54mm
- R1, R10, R11, R12, R13, R14, R15, R16, R17, R18, R19, R2, R20, R21, R22, R23, R24, R25, R26, R27, R28, R29, R3, R30, R31, R32, R33, R34, R35, R36, R37, R38, R39, R4, R40, R5, R6, R7, R8, R9: footprint (none) -> Resistors_THT:R_Axial_DIN0204_L3.6mm_D1.6mm_P5.08mm_Horizontal
- R41, R42, R43, R44, R45, R46, R47, R48, R49, R50, R51, R52, R53, R54, R55, R56, R57, R58, R59, R60: footprint (none) -> Resistors_SMD:R_0805
- R85, R86, R87: renamed from R?; footprint (none) -> Resistors_SMD:R_0805
- SW1: renamed from SW?; footprint nhantt-kicad-lib:button-pcb-10mm -> Buttons_Switches_SMD:SW_DIP_x1_W5.08mm_Slide_Copal_CHS-A
- U10: footprint TQFP100 -> Housings_QFP:LQFP-100_14x14mm_Pitch0.5mm
- U6, U7, U8, U9: footprint (none) -> Housings_DIP:DIP-14_W7.62mm
Connections:
- net 1: no longer U6.3
- net 10: no longer U7.9
- net 11: no longer U7.11
- net 12: no longer U8.1
- net 13: no longer U7.13
- net 14: no longer U8.3
- net 15: no longer U8.5
- net 16: no longer U8.9
- net 17: no longer U8.11
- net 18: no longer U9.3
- net 19: no longer U8.13
- net 2: no longer U6.1
- net 20: no longer U9.1
- net 3: no longer U6.5
- net 4: no longer U6.11
- net 5: no longer U6.13
- net 6: no longer U6.9
- net 7: no longer U7.1
- net 8: no longer U7.3
- net 9: no longer U7.5
- net GND: now also R61.1, R62.1, R63.1, R64.1, R65.1, R66.1, R67.1, R68.1, R69.1, R70.1, R71.1, R72.1, R73.1, R74.1, R75.1, R76.1, R77.1, R78.1, R80.1
- net VCC: now also U11.1, U11.3, U11.5, U11.7, U12.1, U12.3, U12.5, U12.7, U13.1, U13.3, U13.5, U13.7, U14.1, U14.3, U14.5, U14.7
- net at C27.2, R87.2, U10.33 (XTAL2): now also Y1.2
- net at C28.1, R87.1, U10.34 (XTAL1): now also Y1.1
- net 37: now reaches U10.53 ((A8)PC0)
- net 37: now also R81.1
- net 36: now reaches U10.54 ((A9)PC1)
- net 36: now also R103.1
- net 35: now reaches U10.55 ((A10)PC2)
- net 35: now also R83.1
- net 34: now reaches U10.56 ((A11)PC3)
- net 34: now also R107.1
- net 33: now reaches U10.57 ((A12)PC4)
- net 33: now also R144.1
- net 32: now reaches U10.58 ((A13)PC5)
- net 32: now also R84.1
- net 31: now reaches U10.59 ((A14)PC6)
- net 31: now also R102.1
- net 30: now reaches U10.60 ((A15)PC7)
- net 30: now also R82.1
- net 29: now reaches U10.71 ((AD7)PA7)
- net 29: now also R124.1
- net 28: now reaches U10.72 ((AD6)PA6)
- net 28: now also R123.1
- net 27: now reaches U10.73 ((AD5)PA5)
- net 27: now also R122.1
- net 26: now reaches U10.74 ((AD4)PA4)
- net 26: now also R121.1
- net 25: now reaches U10.75 ((AD3)PA3)
- net 25: now also R120.1
- net 24: now reaches U10.76 ((AD2)PA2)
- net 24: now also R125.1
- net 23: now reaches U10.77 ((AD1)PA1)
- net 23: now also R101.1
- net 22: now reaches U10.78 ((AD0)PA0)
- net 22: now also R100.1
- new net: R108.2, R109.2, R110.2, U12.16
- new net: R100.2, U12.2
- new net: Q7.3 (S), U12.13
- new net: R111.2, R112.2, R113.2, U12.14
- new net: R101.2, U12.4
- new net: R141.2, R142.2, R143.2, U14.12
- new net: R125.2, U14.6
- new net: R126.2, R127.2, R128.2, U13.14
- new net: R120.2, U13.4
- new net: R129.2, R130.2, R131.2, U13.12
- new net: R121.2, U13.6
- new net: R132.2, R133.2, R134.2, U13.10
- new net: R122.2, U13.8
- new net: R135.2, R136.2, R137.2, U14.16
- new net: R123.2, U14.2
- new net: R138.2, R139.2, R140.2, U14.14
- new net: R124.2, U14.4
- new net: R91.2, R92.2, R93.2, U11.14
- new net: R82.2, U11.4
- new net: R114.2, R115.2, R116.2, U12.12
- new net: R102.2, U12.6
- new net: R97.2, R98.2, R99.2, U11.10
- new net: R84.2, U11.8
- new net: R145.2, R146.2, R147.2, U14.10
- new net: R144.2, U14.8
- new net: R104.2, R105.2, R106.2, U13.16
- new net: R107.2, U13.2
- new net: R94.2, R95.2, R96.2, U11.12
- new net: R83.2, U11.6
- new net: R117.2, R118.2, R119.2, U12.10
- new net: R103.2, U12.8
- new net: R88.2, R89.2, R90.2, U11.16
- new net: R81.2, U11.2
- new net: D1.1 (K), R61.2
- new net: D2.1 (K), R62.2
- new net: D3.1 (K), R63.2
- new net: D4.1 (K), R64.2
- new net: D5.1 (K), R65.2
- new net: D6.1 (K), R66.2
- new net: D7.1 (K), R67.2
- new net: D8.1 (K), R68.2
- new net: D9.1 (K), R69.2
- new net: D10.1 (K), R70.2
- new net: D11.1 (K), R71.2
- new net: D12.1 (K), R72.2
- new net: D13.1 (K), R73.2
- new net: D14.1 (K), R74.2
- new net: D15.1 (K), R75.2
- new net: D16.1 (K), R76.2
- new net: D17.1 (K), R77.2
- new net: D18.1 (K), R78.2
- new net: D19.1 (K), R79.2
- new net: D20.1 (K), R80.2
- new net: D28.2 (A), J12.2 (Pin_2), Q7.1 (D)
- new net: Q7.2 (G), R113.1
- new net: D36.2 (A), J20.2 (Pin_2), Q15.1 (D)
- new net: Q15.2 (G), R143.1
- new net: D31.2 (A), J15.2 (Pin_2), Q10.1 (D)
- new net: Q10.2 (G), R128.1
- new net: D32.2 (A), J16.2 (Pin_2), Q11.1 (D)
- new net: Q11.2 (G), R131.1
- new net: D33.2 (A), J17.2 (Pin_2), Q12.1 (D)
- new net: Q12.2 (G), R134.1
- new net: D34.2 (A), J18.2 (Pin_2), Q13.1 (D)
- new net: Q13.2 (G), R137.1
- new net: D22.2 (A), J5.2 (Pin_2), Q1.1 (D)
- new net: Q1.2 (G), R90.1
- new net: D29.2 (A), J13.2 (Pin_2), Q8.1 (D)
- new net: Q8.2 (G), R116.1
- new net: D30.2 (A), J14.2 (Pin_2), Q9.1 (D)
- new net: Q9.2 (G), R119.1
- new net: D26.2 (A), J9.2 (Pin_2), Q5.1 (D)
- new net: Q5.2 (G), R106.1
- new net: D23.2 (A), J6.2 (Pin_2), Q2.1 (D)
- new net: Q2.2 (G), R93.1
- new net: D24.2 (A), J7.2 (Pin_2), Q3.1 (D)
- new net: Q3.2 (G), R96.1
- new net: D27.2 (A), J11.2 (Pin_2), Q6.1 (D)
- new net: Q6.2 (G), R110.1
- new net: D25.2 (A), J8.2 (Pin_2), Q4.1 (D)
- new net: Q4.2 (G), R99.1
- new net: D37.2 (A), J21.2 (Pin_2), Q16.1 (D)
- new net: Q16.2 (G), R147.1
- new net: D35.2 (A), J19.2 (Pin_2), Q14.1 (D)
- new net: Q14.2 (G), R140.1
- new net +24V-OUT: D22.1 (K), D23.1 (K), D24.1 (K), D25.1 (K), D26.1 (K), D27.1 (K), D28.1 (K), D29.1 (K), D30.1 (K), D31.1 (K), D32.1 (K), D33.1 (K), D34.1 (K), D35.1 (K), D36.1 (K), D37.1 (K), J10.1 (Pin_1), J11.1 (Pin_1), J12.1 (Pin_1), J13.1 (Pin_1), J14.1 (Pin_1), J15.1 (Pin_1), J16.1 (Pin_1), J17.1 (Pin_1), J18.1 (Pin_1), J19.1 (Pin_1), J20.1 (Pin_1), J21.1 (Pin_1), J5.1 (Pin_1), J6.1 (Pin_1), J7.1 (Pin_1), J8.1 (Pin_1), J9.1 (Pin_1), R104.1, R108.1, R111.1, R114.1, R117.1, R126.1, R129.1, R132.1, R135.1, R138.1, R141.1, R145.1, R88.1, R91.1, R94.1, R97.1
- new net 0V-OUT: J10.2 (Pin_2), Q1.3 (S), Q10.3 (S), Q11.3 (S), Q12.3 (S), Q13.3 (S), Q14.3 (S), Q15.3 (S), Q16.3 (S), Q2.3 (S), Q3.3 (S), Q4.3 (S), Q5.3 (S), Q6.3 (S), Q8.3 (S), Q9.3 (S), R105.1, R109.1, R112.1, R115.1, R118.1, R127.1, R130.1, R133.1, R136.1, R139.1, R142.1, R146.1, R89.1, R92.1, R95.1, R98.1, U11.11, U11.13, U11.15, U11.9, U12.11, U12.15, U12.9, U13.11, U13.13, U13.15, U13.9, U14.11, U14.13, U14.15, U14.9
- new net I1: D1.2 (A), U6.3
- new net I10: D10.2 (A), U7.9
- new net I11: D11.2 (A), U7.11
- new net I12: D12.2 (A), U8.1
- new net I13: D13.2 (A), U7.13
- new net I14: D14.2 (A), U8.3
- new net I15: D15.2 (A), U8.5
- new net I16: D16.2 (A), U8.9
- new net I17: D17.2 (A), U8.11
- new net I18: D18.2 (A), U9.3
- new net I19: D19.2 (A), U8.13
- new net I2: D2.2 (A), U6.1
- new net I20: D20.2 (A), U9.1
- new net I3: D3.2 (A), U6.5
- new net I4: D4.2 (A), U6.11
- new net I5: D5.2 (A), U6.13
- new net I6: D6.2 (A), U6.9
- new net I7: D7.2 (A), U7.1
- new net I8: D8.2 (A), U7.3
- new net I9: D9.2 (A), U7.5

Commit message: sap xep linh kien
Parts:
- R1, R10, R11, R12, R13, R14, R15, R16, R17, R18, R19, R2, R20, R21, R22, R23, R24, R25, R26, R27, R28, R29, R3, R30, R31, R32, R33, R34, R35, R36, R37, R38, R39, R4, R40, R5, R6, R7, R8, R9: footprint Resistors_THT:R_Axial_DIN0204_L3.6mm_D1.6mm_P5.08mm_Horizontal -> Resistors_SMD:R_2512
- R108, R111, R114, R117, R126, R129, R132, R135, R138, R141, R145, R88, R91, R94, R97: value 10K -> 10K/0.6W; footprint Resistors_SMD:R_0805 -> Resistors_SMD:R_2512
- R109, R112, R115, R118, R127, R130, R133, R136, R139, R142, R146, R89, R92, R95, R98: value 1K -> 1K/0.6W; footprint Resistors_SMD:R_0805 -> Resistors_SMD:R_2512
- R110, R113, R116, R119, R128, R131, R134, R137, R140, R143, R90, R93, R96, R99: value 10R -> 10R/0.6W; footprint Resistors_SMD:R_0805 -> Resistors_SMD:R_2512
- R147: value 10R -> 10/R0.6W; footprint Resistors_SMD:R_0805 -> Resistors_SMD:R_2512
- R61, R62, R63, R64, R65, R66, R67, R68, R69, R70, R71, R72, R73, R74, R75, R76, R77, R78, R79, R80: value 220R/0.6W -> 220R; footprint Resistors_THT:R_Axial_DIN0204_L3.6mm_D1.6mm_P5.08mm_Horizontal -> Resistors_SMD:R_0805
Connections:
- net GND: now also R79.1

Commit message: complete
Parts:
- added J22: +5V, Termical-block-2:Pin_Header_Angled_1x02_Pitch2.54mm, symbol Conn_01x02
- added J23, J24, J25: I2C, nhantt-kicad-lib:Pin_Header_Straight_1x04_Pitch2.54mm, symbol Conn_01x04
- added J26: ADC-5V, nhantt-kicad-lib:Pin_Header_Straight_1x10_Pitch2.54mm, symbol Conn_01x10
- added J27: UART, nhantt-kicad-lib:Pin_Header_Straight_1x08_Pitch2.54mm, symbol Conn_01x08
- added P1, P2: CONN_01X01, nhantt-kicad-lib:Vit-3mm, symbol Conn_01x01
- J1: footprint Pin_Headers:Pin_Header_Straight_1x20_Pitch2.54mm -> mods:Terminal-block-20
- J10, J11, J12, J13, J14, J15, J16, J17, J18, J19, J2, J20, J21, J5, J6, J7, J8, J9: footprint Pin_Headers:Pin_Header_Angled_1x02_Pitch2.54mm -> Termical-block-2:Pin_Header_Angled_1x02_Pitch2.54mm
- P10, P11, P12, P13, P8, P9: footprint Pin_Headers:Pin_Header_Angled_1x01_Pitch2.54mm -> nhantt-kicad-lib:Vit-3mm; symbol CONN_01X01 -> Conn_01x01
- R108, R109, R110, R111, R112, R113, R114, R115, R116, R117, R118, R119, R126, R127, R128, R129, R130, R131, R132, R133, R134, R135, R136, R137, R138, R139, R140, R141, R142, R143, R145, R146, R147, R88, R89, R90, R91, R92, R93, R94, R95, R96, R97, R98, R99: footprint Resistors_SMD:R_2512 -> Resistors_SMD:R_0805
- U10: footprint Housings_QFP:LQFP-100_14x14mm_Pitch0.5mm -> Housings_QFP:TQFP-100_14x14mm_Pitch0.5mm
Connections:
- net labels added: 2/INT4, 3/INT5, RX1, RX2, RX3, SCL, SDA, TX1, TX2, TX3
- net labels removed: 1, 14, 15, 16, 17, 18, 19, 2, 20, 3
- wire segments 630 -> 662
- no-connect marks 6 -> 0
Other:
- moved on the sheet: D26, D27, D28, D29, D30, D31, D32, D33, D34, D35, D36, D37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
